Commit message: Added static camera to husky model

File: husky_ws/src/husky_custom_description/urdf/custom_description.urdf.xacro (robot description, xacro)
@@ -46,3 +46,9 @@
   </joint>
   <link name="bumblebee"/>
+  <joint name="arch_to_axis_base" type="fixed">
+    <parent link="arch"/>
+    <child link="axis_base"/>
+    <origin xyz="0.1 -0.20 0.55" rpy="0.0 0.0 0.0" />
+  </joint>
+  <link name="axis_base" />
 </robot>

File: husky_ws/src/husky_custom_gazebo/urdf/custom_description.gazebo.xacro (robot description, xacro)
@@ -90,3 +90,43 @@
     </sensor>
   </gazebo>
+  <!-- camera -->
+   <gazebo reference="axis_base">
+     <sensor type="camera" name="axis_camera">
+       <update_rate>30.0</update_rate>
+       <camera name="head">
+         <horizontal_fov>1.3962634</horizontal_fov>
+         <image>
+           <width>800</width>
+           <height>800</height>
+           <format>R8G8B8</format>
+         </image>
+         <clip>
+           <near>0.02</near>
+           <far>300</far>
+         </clip>
+         <noise>
+           <type>gaussian</type>
+           <!-- Noise is sampled independently per pixel on each frame.
+                That pixel's noise value is added to each of its color
+                channels, which at that point lie in the range [0,1]. -->
+           <mean>0.0</mean>
+           <stddev>0.007</stddev>
+         </noise>
+       </camera>
+       <plugin name="camera_controller" filename="libgazebo_ros_camera.so">
+         <alwaysOn>true</alwaysOn>
+         <updateRate>0.0</updateRate>
+         <cameraName>/axis</cameraName>
+         <imageTopicName>image_raw</imageTopicName>
+         <cameraInfoTopicName>camera_info</cameraInfoTopicName>
+         <frameName>camera_link</frameName>
+         <hackBaseline>0.07</hackBaseline>
+         <distortionK1>0.0</distortionK1>
+         <distortionK2>0.0</distortionK2>
+         <distortionK3>0.0</distortionK3>
+         <distortionT1>0.0</distortionT1>
+         <distortionT2>0.0</distortionT2>
+       </plugin>
+     </sensor>
+   </gazebo>
 </robot>

Commit message: Added that husky navigation launch file, added initial ptz control node

File: husky_ws/src/husky_custom_description/urdf/custom_description.urdf.xacro (robot description, xacro)
@@ -43,5 +43,5 @@
      <parent link="arch"/>
      <child link="bumblebee"/>
-     <origin xyz="0.0 0.0 0.42" rpy="0.0 0.0 0.0"/>
+     <origin xyz="0.0 0.0 0.42" rpy="-1.57079632679 0.0 -1.57079632679"/>
   </joint>
   <link name="bumblebee"/>
